Commit message: Spawned robot in gazebo + added wheels + added plugin to move it in gazebo

File: urdf/erl1.urdf (robot description, URDF)
Before this commit: robot erl1, 1 links, 0 joints
Links:
- added link left_wheel, mass 5.0; collision cylinder length=.05 radius=.1; visual cylinder length=.05 radius=.1
- added link right_wheel, mass 5.0; collision cylinder length=.05 radius=.1; visual cylinder length=.05 radius=.1
Joints:
- added joint left_wheel_joint: type continuous, parent link_chassis, child left_wheel, origin xyz=-0.1 0.15 0 rpy=0 0 0, axis 0 1 0, limit effort=100 velocity=10
- added joint right_wheel_joint: type continuous, parent link_chassis, child right_wheel, origin xyz=-0.1 -0.15 0 rpy=0 0 0, axis 0 1 0, limit effort=100 velocity=10

Commit message: Modification for MOGI robot simulation

File: urdf/erl1.urdf (robot description, URDF)
Before this commit: robot erl1, 5 links, 4 joints
Links:
- removed link link_arm
- removed link link_cube
- link link_chassis: geometry collision mesh filename=package://erl1/meshes/mogi_bot.dae; collision sphere radius=0.05
Joints:
- removed joint arm_joint
- removed joint cube_joint

Commit message: Added lidar

File: urdf/erl1.urdf (robot description, URDF)
Before this commit: robot erl1, 7 links, 6 joints
Links:
- added link scan_link, mass 1e-5; collision box size=.1 .1 .1; visual mesh filename=package://bme_gazebo_sensors/meshes/lidar.dae
Joints:
- added joint scan_joint: type fixed, parent base_link, child scan_link, axis 0 1 0

Commit message: Removed dependency from erl1_sensor pkg

File: urdf/erl1.urdf (robot description, URDF)
Before this commit: robot erl1, 8 links, 7 joints
Links:
- removed link link_chassis
- removed link scan_link
- added link base_footprint
- added link base_link, mass 15.0; collision box size=.4 .2 .1; collision sphere radius=0.0499
- link left_wheel: geometry collision cylinder length=.05 radius=.1; visual mesh filename=package://erl1/meshes/wheel.dae
- link right_wheel: geometry collision cylinder length=.05 radius=.1; visual mesh filename=package://erl1/meshes/wheel.dae
Joints:
- removed joint scan_joint
- added joint base_footprint_joint: type fixed, parent base_footprint, child base_link, origin xyz=0 0 0 rpy=0 0 0
- joint left_wheel_joint: origin xyz=-0.1 0.15 0 rpy=0 0 0 -> xyz=0 0.15 0 rpy=0 0 0; parent link_chassis -> base_link
- joint right_wheel_joint: origin xyz=-0.1 -0.15 0 rpy=0 0 0 -> xyz=0 -0.15 0 rpy=0 0 0; parent link_chassis -> base_link

Commit message: Implemented skid-steering drive with 4 wheels

File: urdf/erl1.urdf (robot description, URDF)
Before this commit: robot erl1, 8 links, 7 joints
Links:
- removed link left_wheel
- removed link right_wheel
- added link left_front_wheel, mass 5.0; collision cylinder length=.05 radius=.1; visual mesh filename=package://erl1/meshes/wheel.dae
- added link left_rear_wheel, mass 5.0; collision cylinder length=.05 radius=.1; visual mesh filename=package://erl1/meshes/wheel.dae
- added link right_front_wheel, mass 5.0; collision cylinder length=.05 radius=.1; visual mesh filename=package://erl1/meshes/wheel.dae
- added link right_rear_wheel, mass 5.0; collision cylinder length=.05 radius=.1; visual mesh filename=package://erl1/meshes/wheel.dae
Joints:
- removed joint left_wheel_joint
- removed joint right_wheel_joint
- added joint left_front_wheel_joint: type continuous, parent base_link, child left_front_wheel, origin xyz=0.15 0.15 0 rpy=0 0 0, axis 0 1 0, limit effort=100 velocity=10
- added joint left_rear_wheel_joint: type continuous, parent base_link, child left_rear_wheel, origin xyz=-0.15 0.15 0 rpy=0 0 0, axis 0 1 0, limit effort=100 velocity=10
- added joint right_front_wheel_joint: type continuous, parent base_link, child right_front_wheel, origin xyz=0.15 -0.15 0 rpy=0 0 0, axis 0 1 0, limit effort=100 velocity=10
- added joint right_rear_wheel_joint: type continuous, parent base_link, child right_rear_wheel, origin xyz=-0.15 -0.15 0 rpy=0 0 0, axis 0 1 0, limit effort=100 velocity=10

Commit message: Removed casters

File: urdf/erl1.urdf (robot description, URDF)
Before this commit: robot erl1, 10 links, 9 joints
Links:
- link base_link: geometry collision box size=.4 .2 .1; visual mesh filename=package://erl1/meshes/mogi_bot.dae
